File: gnat-1.brd (EAGLE design)
At the start: 58.5 x 25.1 mm, 25 parts, among them IC1 ATMEGA, IC2 MCP1702-33, J1 USB-A-H, X1 16 MHz

Commit message: update
Parts:
- removed J6: (no value), SparkFun-Connectors:1X12
- removed J9: (no value), SparkFun-Connectors:SCREWTERMINAL-3.5MM-4
- removed JP2: (no value), pinhead:2X05
- removed JP3, JP4: (no value), pinhead:2X06
- added C7: 0.1µ, resistor:C025-024X044
- added R3, R4: 10k, resistor:0204/7
- J2: device SparkFun-Connectors:1X06 -> SparkFun-Connectors:1X04
- J3: device SparkFun-Connectors:1X02 -> SparkFun-Connectors:1X06
- J4: device SparkFun-Connectors:1X08_ROUND -> SparkFun-Connectors:1X06
- J5: device SparkFun-Connectors:SCREWTERMINAL-3.5MM-3 -> SparkFun-Connectors:1X02
- moved J5 42.3 mm to (39.8, 15.0), turned to 0 degrees
- moved J2 28.9 mm to (34.6, 12.4), turned to 0 degrees
- moved C2 27.0 mm to (53.8, 5.94)
- moved R2 20.9 mm to (18.5, 12.0), turned to 180 degrees
- moved J4 8.75 mm to (7.95, 23.8)
- moved IC2 7.34 mm to (11.4, 13.7), turned to 270 degrees
- moved C4 7.04 mm to (16.1, 16.1), turned to 180 degrees
- moved R1 6.47 mm to (16.6, 18.6)
- moved C3 5.16 mm to (8.11, 13.6), turned to 90 degrees
- moved J3 4.52 mm to (7.95, 21.2), turned to 0 degrees
- moved C1 3.84 mm to (9.42, 17.9)
- moved C5 2.72 mm to (26.3, 16.2), turned to 180 degrees
- moved IC1 0.49 mm to (25.3, 5.79), turned to 180 degrees
- moved ISP 0.38 mm to (48.4, 4.11)
- moved X1 0.16 mm to (29.0, 12.8), turned to 0 degrees
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Connections:
- removed net MISO: ISP.1
- removed net MOSI: ISP.4
- removed net RESET: ISP.5
- removed net SCK: ISP.3
- removed net VBUS: ISP.2
- new net N$3: J2.1, JP1.EARTH
- new net N$4: J2.2, JP1.RING1
- new net N$5: J2.3, JP1.TIP
- new net N$6: J2.4, JP1.RING2
- new net N$7: C7.2, R3.2, R4.2
- new net N$8: J5.1, R4.1
- net A0: now also J8.2
- net A1: now also J8.1
- net A2: now also J4.5
- net A3: now also J4.4
- net A4_SDA: now also J7.2
- net A5_SCL: now also J7.1
- net D0_RX: now also J3.4; no longer J2.4
- net D11_MOSI: now also ISP.4
- net D12_MISO: now also ISP.1
- net D13_SCK: now also ISP.3
- net D1_TX: now also J3.5; no longer J2.5
- net D2: now also J4.6
- net D3: now also C7.1
- net D4: now also J4.3
- net D5: now also J4.2
- net GND: now also J3.1, J4.1, J5.2, J7.3, J8.3, R3.1; no longer J2.1, J3.2
- net N$20: now also J3.6; no longer J2.6
- net PWR: now also ISP.2, J3.3; no longer J2.3, J3.1
- net RST: now also ISP.5
- net VCC: now also J7.4, J8.4
Other:
- board text removed: "3.3"
- board text removed: "A0"
- board text removed: "A1"
- board text removed: "A2"
- board text removed: "A3"
- board text removed: "A4"
- board text removed: "A5"
- board text removed: "AREF"
- board text removed: "C1"
- board text removed: "C2"
- board text removed: "C3"
- board text removed: "C4"
- board text removed: "C5"
- board text removed: "D10"
- board text removed: "D11"
- board text removed: "D12"
- board text removed: "D13"
- board text removed: "D2"
- board text removed: "D3"
- board text removed: "D4"
- board text removed: "D5"
- board text removed: "D6"
- board text removed: "D7"
- board text removed: "D8"
- board text removed: "D9"
- board text removed: "DTR"
- board text removed: "E1"
- board text removed: "E2"
- board text removed: "E3"
- board text removed: "E4"
- board text removed: "E5"
- board text removed: "E6"
- board text removed: "E7"
- board text removed: "E8"
- board text removed: "GND"
- board text removed: "IC1"
- board text removed: "IC2"
- board text removed: "LED"
- board text removed: "NC"
- board text removed: "R1"
- board text removed: "R2"
- board text removed: "RST"
- board text removed: "RX"
- board text removed: "TX"
- board text removed: "VIN"
- board text removed: "X1"
- board text removed: "X3"
