File: gnat-1.sch (EAGLE design)
At the start: 25 parts, among them IC1 ATMEGA, IC2 MCP1702-33, J1 USB-A-H, X1 16 MHz

Commit message: update
Parts:
- removed J6: (no value), SparkFun-Connectors:M12PTH
- removed J9: (no value), SparkFun-Connectors:M04SCREW
- removed JP2: (no value), pinhead:PINHD-2X5
- removed JP3, JP4: (no value), pinhead:PINHD-2X6
- added C7: 0.1µ, resistor:C-EU025-024X044
- added R3, R4: 10k, resistor:R-EU_0204/7
- J2: device SparkFun-Connectors:M06SILK_FEMALE_PTH -> SparkFun-Connectors:M04PTH
- J3: device SparkFun-Connectors:M02PTH -> SparkFun-Connectors:M06SILK_FEMALE_PTH
- J4: device SparkFun-Connectors:M08 -> SparkFun-Connectors:M06SILK_FEMALE_PTH
- J5: device SparkFun-Connectors:M03SCREW -> SparkFun-Connectors:M02PTH
Connections:
- removed net MISO: ISP.1
- removed net MOSI: ISP.4
- removed net RESET: ISP.5
- removed net SCK: ISP.3
- removed net VBUS: ISP.2
- new net N$3: J2.1, JP1.EARTH
- new net N$4: J2.2, JP1.RING1
- new net N$5: J2.3, JP1.TIP
- new net N$6: J2.4, JP1.RING2
- new net N$7: C7.2, R3.2, R4.2
- new net N$8: J5.1, R4.1
- net A0: now also J8.2
- net A1: now also J8.1
- net A2: now also J4.5
- net A3: now also J4.4
- net A4_SDA: now also J7.2
- net A5_SCL: now also J7.1
- net D0_RX: now also J3.4; no longer J2.4
- net D11_MOSI: now also ISP.4
- net D12_MISO: now also ISP.1
- net D13_SCK: now also ISP.3
- net D1_TX: now also J3.5; no longer J2.5
- net D2: now also J4.6
- net D3: now also C7.1
- net D4: now also J4.3
- net D5: now also J4.2
- net GND: now also J3.1, J4.1, J5.2, J7.3, J8.3, R3.1; no longer J2.1, J3.2
- net N$20: now also J3.6; no longer J2.6
- net PWR: now also ISP.2, J3.3; no longer J2.3, J3.1
- net RST: now also ISP.5
- net VCC: now also J7.4, J8.4
Other:
- moved on the sheet: ISP, J7, J8, JP1
